File: hardware/processor.sch (KiCad schematic (older format))
At the start: 22 parts, among them J1 USB_2, P3 CONN_3X2, U10 ATMEGA32U4, U9 USB6B1, X2 16 MHz

Commit message: updated schematics to include new library and added uSD drive to processor
Parts:
- removed U9: USB6B1, symbol USB6B1
- added R? (x8): DNI, symbol R
- added U?: CONN_MICROSD, symbol CONN_MICROSD
Connections:
- net labels removed: spi_clk
- wire segments 94 -> 156
Other:
- note added: "3M 290805\nDigi-Key 3M5607CT-NO\n"
- moved on the sheet: C22, C23, C24, C25, C26, C27, C28, C29, C30, D10, D9, J1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
