File: hardware/can.sch (KiCad schematic (older format))
At the start: 17 parts, among them U4 MCP2515, U5 MCP2551_1, X1 20 MHz

Commit message: fixed some ERCs and simplified reset
Parts:
- renumbered C13 to C15, C14 to C16, C15 to C17, C16 to C18, C17 to C19, C18 to C20, D3 to D6, D4 to D7, R14 to R13, R15 to R14, R16 to R15, R17 to R16, R18 to R17, R19 to R18, U4 to U5, U5 to U6
Changed lines of the file:
@@
-EESchema Schematic File Version 2  date Sat 26 Apr 2014 10:24:32 PM EDT
+EESchema Schematic File Version 2  date Wed 30 Apr 2014 02:36:15 PM EDT
 LIBS:power
 LIBS:device
@@
 Sheet 4 6
 Title ""
-Date "27 apr 2014"
+Date "30 apr 2014"
 Rev ""
 Comp ""
@@
 Connection ~ 6200 2300
 $Comp
-L MCP2551_1 U5
+L MCP2551_1 U6
 U 1 1 5277CB7E
 P 7450 4000
-F 0 "U5" H 7450 3950 60  0000 C CNN
+F 0 "U6" H 7450 3950 60  0000 C CNN
 F 1 "MCP2551_1" H 7400 4050 60  0000 C CNN
 	1    7450 4000
@@
 NoConn ~ 3400 4050
 $Comp
-L +5V #PWR012
+L +5V #PWR014
 U 1 1 527292FD
 P 5250 2200
-F 0 "#PWR012" H 5250 2290 20  0001 C CNN
+F 0 "#PWR014" H 5250 2290 20  0001 C CNN
 F 1 "+5V" H 5250 2290 30  0000 C CNN
 	1    5250 2200
@@
 $EndComp
 $Comp
-L R R15
+L R R14
 U 1 1 527292F3
 P 5550 2650
-F 0 "R15" V 5630 2650 50  0000 C CNN
+F 0 "R14" V 5630 2650 50  0000 C CNN
 F 1 "1k" V 5550 2650 50  0000 C CNN
 	1    5550 2650
@@
 $EndComp
 $Comp
-L R R14
+L R R13
 U 1 1 527292E1
 P 5250 2650
-F 0 "R14" V 5330 2650 50  0000 C CNN
+F 0 "R13" V 5330 2650 50  0000 C CNN
 F 1 "1k" V 5250 2650 50  0000 C CNN
 	1    5250 2650
@@
 $EndComp
 $Comp
-L LED D4
+L LED D7
 U 1 1 527292D6
 P 5550 3250
-F 0 "D4" H 5550 3350 50  0000 C CNN
+F 0 "D7" H 5550 3350 50  0000 C CNN
 F 1 "LED" H 5550 3150 50  0000 C CNN
 	1    5550 3250
@@
 $EndComp
 $Comp
-L LED D3
+L LED D6
 U 1 1 527292B1
 P 5250 3250
-F 0 "D3" H 5250 3350 50  0000 C CNN
+F 0 "D6" H 5250 3350 50  0000 C CNN
 F 1 "LED" H 5250 3150 50  0000 C CNN
 	1    5250 3250
@@
 $EndComp
 $Comp
-L +5V #PWR013
+L +5V #PWR015
 U 1 1 527287C3
 P 4150 3200
-F 0 "#PWR013" H 4150 3290 20  0001 C CNN
+F 0 "#PWR015" H 4150 3290 20  0001 C CNN
 F 1 "+5V" H 4150 3290 30  0000 C CNN
 	1    4150 3200
@@
 $EndComp
 $Comp
-L +5V #PWR014
+L +5V #PWR016
 U 1 1 526D809E
 P 2450 5700
-F 0 "#PWR014" H 2450 5790 20  0001 C CNN
+F 0 "#PWR016" H 2450 5790 20  0001 C CNN
 F 1 "+5V" H 2450 5790 30  0000 C CNN
 	1    2450 5700
@@
 $EndComp
 $Comp
-L GND #PWR015
+L GND #PWR017
 U 1 1 526D809D
 P 2450 6300
-F 0 "#PWR015" H 2450 6300 30  0001 C CNN
+F 0 "#PWR017" H 2450 6300 30  0001 C CNN
 F 1 "GND" H 2450 6230 30  0001 C CNN
 	1    2450 6300
@@
 $EndComp
 $Comp
-L C C16
+L C C18
 U 1 1 526D809C
 P 2450 6000
-F 0 "C16" H 2500 6100 50  0000 L CNN
+F 0 "C18" H 2500 6100 50  0000 L CNN
 F 1 "0.1 uF" H 2500 5900 50  0000 L CNN
 	1    2450 6000
@@
 $EndComp
 $Comp
-L C C15
+L C C17
 U 1 1 526D8053
 P 2100 6000
-F 0 "C15" H 2150 6100 50  0000 L CNN
+F 0 "C17" H 2150 6100 50  0000 L CNN
 F 1 "0.1 uF" H 2150 5900 50  0000 L CNN
 	1    2100 6000
@@
 $EndComp
 $Comp
-L GND #PWR016
+L GND #PWR018
 U 1 1 526D8048
 P 2100 6300
-F 0 "#PWR016" H 2100 6300 30  0001 C CNN
+F 0 "#PWR018" H 2100 6300 30  0001 C CNN
 F 1 "GND" H 2100 6230 30  0001 C CNN
 	1    2100 6300
@@
 $EndComp
 $Comp
-L GND #PWR017
+L GND #PWR019
 U 1 1 52653C19
 P 8800 5400
-F 0 "#PWR017" H 8800 5400 30  0001 C CNN
+F 0 "#PWR019" H 8800 5400 30  0001 C CNN
 F 1 "GND" H 8800 5330 30  0001 C CNN
 	1    8800 5400
@@
 $EndComp
 $Comp
-L C C18
+L C C20
 U 1 1 52653BFD
 P 9150 4850
-F 0 "C18" H 9200 4950 50  0000 L CNN
+F 0 "C20" H 9200 4950 50  0000 L CNN
 F 1 "560 pF" H 9200 4750 50  0000 L CNN
 	1    9150 4850
@@
 $EndComp
 $Comp
-L C C17
+L C C19
 U 1 1 52653BE2
 P 8800 4850
-F 0 "C17" H 8850 4950 50  0000 L CNN
+F 0 "C19" H 8850 4950 50  0000 L CNN
 F 1 "560 pF" H 8850 4750 50  0000 L CNN
 	1    8800 4850
@@
 $EndComp
 $Comp
-L R R19
+L R R18
 U 1 1 52653BCF
 P 9150 4300
-F 0 "R19" V 9230 4300 50  0000 C CNN
+F 0 "R18" V 9230 4300 50  0000 C CNN
 F 1 "100" V 9150 4300 50  0000 C CNN
 	1    9150 4300
@@
 $EndComp
 $Comp
-L R R18
+L R R17
 U 1 1 52653BC8
 P 8800 4300
-F 0 "R18" V 8880 4300 50  0000 C CNN
+F 0 "R17" V 8880 4300 50  0000 C CNN
 F 1 "100" V 8800 4300 50  0000 C CNN
 	1    8800 4300
@@
 $EndComp
 $Comp
-L R R16
+L R R15
 U 1 1 5265384F
 P 6200 4250
-F 0 "R16" V 6280 4250 50  0000 C CNN
+F 0 "R15" V 6280 4250 50  0000 C CNN
 F 1 "2k" V 6200 4250 50  0000 C CNN
 	1    6200 4250
@@
 can_h
 $Comp
-L R R17
+L R R16
 U 1 1 526534F5
 P 6500 4650
-F 0 "R17" V 6580 4650 50  0000 C CNN
+F 0 "R16" V 6580 4650 50  0000 C CNN
 F 1 "1K" V 6500 4650 50  0000 C CNN
 	1    6500 4650
@@
 $EndComp
 $Comp
-L GND #PWR018
+L GND #PWR020
 U 1 1 52653459
 P 1050 3850
-F 0 "#PWR018" H 1050 3850 30  0001 C CNN
+F 0 "#PWR020" H 1050 3850 30  0001 C CNN
 F 1 "GND" H 1050 3780 30  0001 C CNN
 	1    1050 3850
@@
 $EndComp
 $Comp
-L C C13
+L C C15
 U 1 1 52653347
 P 1450 2750
-F 0 "C13" H 1500 2850 50  0000 L CNN
+F 0 "C15" H 1500 2850 50  0000 L CNN
 F 1 "C" H 1500 2650 50  0000 L CNN
 	1    1450 2750
@@
 $EndComp
 $Comp
-L C C14
+L C C16
 U 1 1 52653340
 P 1450 3600
-F 0 "C14" H 1500 3700 50  0000 L CNN
+F 0 "C16" H 1500 3700 50  0000 L CNN
 F 1 "C" H 1500 3500 50  0000 L CNN
 	1    1450 3600
@@
 $EndComp
 $Comp
-L +5V #PWR019
+L +5V #PWR021
 U 1 1 52653250
 P 2100 5700
-F 0 "#PWR019" H 2100 5790 20  0001 C CNN
+F 0 "#PWR021" H 2100 5790 20  0001 C CNN
 F 1 "+5V" H 2100 5790 30  0000 C CNN
 	1    2100 5700
@@
 $EndComp
 $Comp
-L GND #PWR020
+L GND #PWR022
 U 1 1 52653212
 P 7450 5300
-F 0 "#PWR020" H 7450 5300 30  0001 C CNN
+F 0 "#PWR022" H 7450 5300 30  0001 C CNN
 F 1 "GND" H 7450 5230 30  0001 C CNN
 	1    7450 5300
@@
 $EndComp
 $Comp
-L GND #PWR021
+L GND #PWR023
 U 1 1 5265320A
 P 4150 5450
-F 0 "#PWR021" H 4150 5450 30  0001 C CNN
+F 0 "#PWR023" H 4150 5450 30  0001 C CNN
 F 1 "GND" H 4150 5380 30  0001 C CNN
 	1    4150 5450
@@
 $EndComp
 $Comp
-L MCP2515 U4
+L MCP2515 U5
 U 1 1 5264697B
 P 4150 4400
-F 0 "U4" H 4150 4350 60  0000 C CNN
+F 0 "U5" H 4150 4350 60  0000 C CNN
 F 1 "MCP2515" H 4150 4450 60  0000 C CNN
 	1    4150 4400
