File: hardware/eng_mon.sch (KiCad schematic (older format))
At the start: 1 part, among them P1 CONN_12

Commit message: updated schematics to include new library and added uSD drive to processor
Changed lines of the file:
@@
-EESchema Schematic File Version 2  date Tue 04 Mar 2014 01:13:50 PM EST
+EESchema Schematic File Version 2  date Sat 26 Apr 2014 10:24:32 PM EDT
 LIBS:power
 LIBS:device
@@
 LIBS:valves
 LIBS:gs
+LIBS:opendous
 LIBS:eng_mon-cache
 EELAYER 25  0
@@
 Sheet 1 6
 Title ""
-Date "4 mar 2014"
+Date "27 apr 2014"
 Rev ""
 Comp ""
@@
 	8250 5900 7200 5900
 Wire Wire Line
-	2000 2150 1600 2150
+	2000 2150 1850 2150
+Wire Wire Line
+	1850 2150 1600 2150
 Wire Wire Line
 	1600 2150 1600 1350
@@
 	5850 3900 4450 3900
 Wire Wire Line
-	3000 2300 5300 2300
+	3000 2300 3150 2300
+Wire Wire Line
+	3150 2300 5300 2300
 Wire Wire Line
 	5300 2300 5300 3400

Commit message: fixed some ERCs and simplified reset
Changed lines of the file:
@@
-EESchema Schematic File Version 2  date Sat 26 Apr 2014 10:24:32 PM EDT
+EESchema Schematic File Version 2  date Wed 30 Apr 2014 02:36:15 PM EDT
 LIBS:power
 LIBS:device
@@
 Sheet 1 6
 Title ""
-Date "27 apr 2014"
+Date "30 apr 2014"
 Rev ""
 Comp ""
@@
 	8250 5900 7200 5900
 Wire Wire Line
-	2000 2150 1850 2150
-Wire Wire Line
-	1850 2150 1600 2150
+	2000 2150 1600 2150
 Wire Wire Line
 	1600 2150 1600 1350
@@
 	5850 3900 4450 3900
 Wire Wire Line
-	3000 2300 3150 2300
-Wire Wire Line
-	3150 2300 5300 2300
+	3000 2300 5300 2300
 Wire Wire Line
 	5300 2300 5300 3400
